Commit message: Add imu_corrector to fix accelerometer readings w/r to the body. Refactor variable & object names for consistency

File: src/uuv_description/urdf/uuv.urdf.xacro (robot description, xacro)
@@ -13,5 +13,5 @@
             <!-- IMU -->
             <link name="imu_link"/>
-            <joint name="base_to_imu" type="fixed">
+            <joint name="fc_to_imu" type="fixed">
                 <parent link="fc_link"/>
                 <child link="imu_link"/>
@@ -20,5 +20,5 @@
             <!-- Compass -->
             <link name="compass_link"/>
-            <joint name="base_to_compass" type="fixed">
+            <joint name="fc_to_compass" type="fixed">
                 <parent link="fc_link"/>
                 <child link="compass_link"/>
@@ -27,5 +27,5 @@
             <!-- Magnetometer -->
             <link name="mag_link"/>
-            <joint name="base_to_mag" type="fixed">
+            <joint name="fc_to_mag" type="fixed">
                 <parent link="fc_link"/>
                 <child link="mag_link"/>
@@ -34,5 +34,5 @@
             <!-- Int. Barometer -->
             <link name="baro_int_link"/>
-            <joint name="base_to_baro_int" type="fixed">
+            <joint name="fc_to_baro_int" type="fixed">
                 <parent link="fc_link"/>
                 <child link="baro_int_link"/>
